File: Block Diagram.kicad_sch (KiCad schematic)
At the start: 0 parts

Commit message: Finished board design, outputs generated
Other:
- note added: "(+3V3 or +5V) VDD"
- note added: "Jumper selector"
- note added: "VDD"
- note removed: "+??V"
- note removed: "+A3V3"
