File: Project Architecture.kicad_sch (KiCad schematic)
At the start: 0 parts

Commit message: Finished board design, outputs generated
Changed lines of the file:
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@@
 		)
 	)
-	(text_box "Description"
+	(text_box "Complete board"
 		(exclude_from_sim no)
 		(at 176.53 54.61 0)
@@
 		(stroke
 			(width -0.0001)
-			(type default)
+			(type solid)
 		)
 		(fill
