File: Revision History.kicad_sch (KiCad schematic)
At the start: 0 parts

Commit message: Finished board design, outputs generated
Changed lines of the file:
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@@
 		)
 	)
-	(text_box "DD.MM.YYYY - xxx Revision\nVariant: xxx"
+	(text_box "26.03.2025 - V2 Revision\nVariant: ${VARIANT}"
 		(exclude_from_sim no)
 		(at 86.36 31.75 0)
@@
 		(stroke
 			(width -0.0001)
-			(type default)
+			(type solid)
 		)
 		(fill
@@
 		)
 	)
-	(text_box "- _________________________________\n\n- _________________________________\n\n- _________________________________\n\n- _________________________________\n\n- _________________________________\n\n- _________________________________\n\n- _________________________________\n\n- _________________________________\n\n- _________________________________\n\n- _________________________________\n\n- _________________________________\n\n- _________________________________\n\n- _________________________________\n\n- _________________________________\n\n- _________________________________\n\n- _________________________________\n\n- _________________________________"
+	(text_box "- First Draft\n\n- Added MCP23017 GPIOs on the header\n\n- Added Jumper selector on LEDs\n\n- Added Output voltage selection\n\n- Added MCP2221 serial on Header\n\n- Added MCP2221 I2C on Header\n\n- _________________________________\n\n- _________________________________\n\n- _________________________________\n\n- _________________________________\n\n- _________________________________\n\n- _________________________________\n\n- _________________________________\n\n- _________________________________\n\n- _________________________________\n\n- _________________________________\n\n- _________________________________"
 		(exclude_from_sim no)
 		(at 22.86 40.64 0)
@@
 		(stroke
 			(width -0.0001)
-			(type default)
+			(type solid)
 		)
 		(fill
@@
 		)
 	)
-	(text_box "DD.MM.YYYY - xxx Revision\nVariant: xxx"
+	(text_box "09.02.2016 - V1 Revision\nVariant: ${VARIANT}"
 		(exclude_from_sim no)
 		(at 20.32 31.75 0)
@@
 		(stroke
 			(width -0.0001)
-			(type default)
+			(type solid)
 		)
 		(fill
@@
 		)
 	)
-	(text_box "- _________________________________\n\n- _________________________________\n\n- _________________________________\n\n- _________________________________\n\n- _________________________________\n\n- _________________________________\n\n- _________________________________\n\n- _________________________________\n\n- _________________________________\n\n- _________________________________\n\n- _________________________________\n\n- _________________________________\n\n- _________________________________\n\n- _________________________________\n\n- _________________________________\n\n- _________________________________\n\n- _________________________________"
+	(text_box "- Changed conmnector to USB-C\n\n- _________________________________\n\n- _________________________________\n\n- _________________________________\n\n- _________________________________\n\n- _________________________________\n\n- _________________________________\n\n- _________________________________\n\n- _________________________________\n\n- _________________________________\n\n- _________________________________\n\n- _________________________________\n\n- _________________________________\n\n- _________________________________\n\n- _________________________________\n\n- _________________________________\n\n- _________________________________"
 		(exclude_from_sim no)
 		(at 88.9 40.64 0)
@@
 		(stroke
 			(width -0.0001)
-			(type default)
+			(type solid)
 		)
 		(fill
