File: IOExtender.kicad_pcb (KiCad board)
At the start: 2 copper layers, 25.6 x 44 mm, 40 parts, among them J1 1x3 pin vertical, J2 1x13, J3 Jumper, J5 1x13, J6 Jumper, J7 Jumper, J8 Jumper, J9 22-28-8083, U1 MCP23017_SS, U2 MCP2221AxSL, U3 NCP1117IST33T3G

Commit message: Finished board design, outputs generated
Parts:
- added TP1: TestPoint, Connector_Pin:Pin_D1.0mm_L10.0mm, B.Cu at (130.6, 94.6)
- added TP2: TestPoint, Connector_Pin:Pin_D1.0mm_L10.0mm, B.Cu at (133.7, 95.9)
- added TP3: TestPoint, Connector_Pin:Pin_D1.0mm_L10.0mm, B.Cu at (136.7, 84.0)
- added TP4: TestPoint, Connector_Pin:Pin_D1.0mm_L10.0mm, B.Cu at (119.7, 96.4)
Routing:
- net +5V: track 14.0 -> 12.9 mm
Other:
- board text added: "+5V +3V3 VDD GND"
- board text added: "0.07mm (2oz)"
- board text added: "0.2000 mm / 0.1500 mm"
- board text added: "0.2500 mm"
- board text added: "0.250mm 0.600mm 1.000mm 0.650mm"
- board text added: "0x40 W 0x41 R"
- board text added: "1.48mm"
- board text added: "1.6600 mm"
- board text added: "130.618 133.666 136.714 119.696"
- board text added: "2"
- board text added: "25.6000 mm x 44.0000 mm"
- board text added: "46 4 slots 41 2"
- board text added: "94.618 95.888 83.95 96.396"
- board text added: "BOARD CHARACTERISTICS"
- board text added: "Board Thickness:"
- board text added: "Board overall dimensions:"
- board text added: "Castellated pads:"
- board text added: "Copper Finish:"
- board text added: "Copper Layer Count:"
- board text added: "Edge card connectors:"
- board text added: "Immersion gold"
- board text added: "Impedance Control:"
- board text added: "Min hole diameter:"
- board text added: "Min track/spacing:"
- board text added: "No"
- board text added: "Plated Board Edge:"
- board text added: "Plated Plated Plated Unplated"
- board text added: "TP1 TP2 TP3 TP4"
- board text added: "Yes"
- board text added: "github: Thiapalm"
- board text removed: "??? ??? ??? ??? ??? (slot) ??? ??? ??? ??? ???"
- board text removed: "???mm"
- board text removed: "???mm (?oz)"
- board text removed: "???mm ???mm ???mm ???mm ???mm ???mm ???mm ???mm ???mm ???mm"
- board text removed: "I2C 0x40 W 0x41 R"
- board text removed: "Internal Plane"
- board text removed: "L3 (Sig, PWR)"
- board text removed: "L4 (Sig, PWR)"
- board text removed: "L5 (GND)"
- board text removed: "L6 (Sig, PWR)"
- board text removed: "PCB3D_BR_BOARDNAME"
- board text removed: "PCB3D_TL_BOARDNAME"
- board text removed: "Plated Plated Plated Plated Plated Plated Plated Plated Plated Unplated"
- board text removed: "Prepreg"

Commit message: Updated Fabrication Files
Parts:
- TP1, TP2, TP3, TP4: footprint Connector_Pin:Pin_D1.0mm_L10.0mm -> 0_testpoints:TestPoint_PTH_1mm_2mm
Other:
- board text added: "17.118 20.166 23.214 6.196"
- board text added: "30.382 29.112 41.159 28.604"
- board text added: "FABRICATION NOTES (UNLESS OTHERWISE SPECIFIED) 1) OUTLINE DEFINED IN SEPARATE GERBER FILE WITH {dblquote}Edge_Cuts.GBR{dblquote} SUFFIX. DIMENSIONS OF CIRCUMSIZED RECTANGLE SHOWN ON THIS DWG FOR REF ONLY. 2) SEE SEPARATE DRILL FILES WITH {dblquote}.DRL{dblquote} SUFFIX FOR HOLE LOCATIONS. SELECTED HOLE LOCATIONS SHOWN ON THIS DWG FOR REF ONLY. 3) CONFIRM TRACE WIDTHS AND SPACINGS. 4) DESIGN GEOME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"
- board text removed: "0.250mm 0.600mm 1.000mm 0.650mm"
- board text removed: "130.618 133.666 136.714 119.696"
- board text removed: "46 4 slots 41 2"
- board text removed: "94.618 95.888 83.95 96.396"
- board text removed: "Count"
- board text removed: "FABRICATION NOTES (UNLESS OTHERWISE SPECIFIED) 1) OUTLINE DEFINED IN SEPARATE GERBER FILE WITH {dblquote}Edge_Cuts.GBR{dblquote} SUFFIX. DIMENSIONS OF CIRCUMSIZED RECTANGLE SHOWN ON THIS DWG FOR REF ONLY. 2) SEE SEPARATE DRILL FILES WITH {dblquote}.DRL{dblquote} SUFFIX FOR HOLE LOCATIONS. SELECTED HOLE LOCATIONS SHOWN ON THIS DWG FOR REF ONLY. 3) IMPEDANCE CONTROL REQUIRED. Microstrip 100-Ohm Dif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"
- board text removed: "Hole Size"
- board text removed: "Plated"
- board text removed: "Plated Plated Plated Unplated"
- board text removed: "Symbol"
