File: Section A - Title A.kicad_sch (KiCad schematic)
At the start: 40 parts, among them J1 1x3 pin vertical, J2 1x13, J3 Jumper, J5 1x13, J6 Jumper, J7 Jumper, J8 Jumper, J9 22-28-8083, U1 MCP23017_SS, U2 MCP2221AxSL, U3 NCP1117IST33T3G

Commit message: Finished board design, outputs generated
Parts:
- added S1: MSA-G, symbol 0_helpers:MSA-G
- added TP1, TP2, TP3, TP4: TestPoint, Connector_Pin:Pin_D1.0mm_L10.0mm, symbol Connector:TestPoint
- C1: Manufacturer Part Number (none) -> C0603C474K3RACTU
- C2: Manufacturer Part Number (none) -> GRM188R61E475KE11D
- C5: Manufacturer Part Number (none) -> USB4215-03-A
- C6: Manufacturer Part Number (none) -> C1608X5R1C106M080AB
- C8: Manufacturer Part Number (none) -> 0805B104K500CT
- D1, D5: Manufacturer Part Number (none) -> LTST-C191KSKT
- D2: Manufacturer Part Number (none) -> SM0603SRC
- D4: Manufacturer Part Number (none) -> CDSOT23-T05LC-Q
- D6, D7: Manufacturer Part Number (none) -> SML-LX0603GW-TR
- J1: Manufacturer Part Number (none) -> G800LR305018EU
- J2, J5: Manufacturer Part Number (none) -> 61301311121
- J9: Manufacturer Part Number (none) -> 22-28-8083
- L1, L2: Manufacturer Part Number (none) -> MPZ2012S331AT000
- R1, R10, R11, R2, R3, R9: Manufacturer Part Number (none) -> CRCW060333R0FKEA
- R12, R13: Manufacturer Part Number (none) -> CRCW06035K10FKEC
- R4, R5, R6, R7, R8: Manufacturer Part Number (none) -> ERJ-3GEYJ331V
- U1: Manufacturer Part Number (none) -> MCP23017_SS
- U2: Manufacturer Part Number (none) -> MCP2221AxSL
- U3: Manufacturer Part Number (none) -> NCP1117IST33T3G
Connections:
- net +3V3: now also TP2.1
- net +5V: now also TP1.1
- net GND: now also TP4.1
- net VDD: now also TP3.1
Other:
- moved on the sheet: J1

Commit message: Updated Fabrication Files
Parts:
- TP1, TP2, TP3, TP4: footprint Connector_Pin:Pin_D1.0mm_L10.0mm -> 0_testpoints:TestPoint_PTH_1mm_2mm
